File: Warsztaty/minisumo/minisumo_pcb/programming_connector.kicad_sch (KiCad schematic)
At the start: 1 part

Commit message: chyba gotowy schemat
Connections:
- net GND: now also SPI1.01; no longer SPI1.06
- net MISO: now also SPI1.06; no longer SPI1.01
Changed lines of the file:
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@@
+	(wire
+		(pts
+			(xy 34.29 30.48) (xy 26.67 30.48)
+		)
+		(stroke
+			(width 0)
+			(type default)
+		)
+	)
+	(wire
+		(pts
+			(xy 26.67 30.48) (xy 26.67 36.83)
+		)
+		(stroke
+			(width 0)
+			(type default)
+		)
+	)
 	(wire
 		(pts
 			(xy 62.23 29.21) (xy 62.23 30.48)
-		)
-		(stroke
-			(width 0)
-			(type default)
-		)
-	)
-	(wire
-		(pts
-			(xy 59.69 35.56) (xy 62.23 35.56)
-		)
-		(stroke
-			(width 0)
-			(type default)
-		)
-	)
-	(wire
-		(pts
-			(xy 62.23 35.56) (xy 62.23 38.1)
 		)
 		(stroke
@@
 		)
 	)
+	(hierarchical_label "MISO"
+		(shape input)
+		(at 59.69 35.56 0)
+		(fields_autoplaced yes)
+		(effects
+			(font
+				(size 0.762 0.762)
+			)
+			(justify left)
+		)
+	)
 	(hierarchical_label "SCK"
 		(shape input)
@@
 			)
 			(justify left)
-		)
-	)
-	(hierarchical_label "MISO"
-		(shape input)
-		(at 34.29 30.48 180)
-		(fields_autoplaced yes)
-		(effects
-			(font
-				(size 0.762 0.762)
-			)
-			(justify right)
 		)
 	)
@@
 	(symbol
 		(lib_id "power:GND")
-		(at 62.23 38.1 0)
+		(at 26.67 36.83 0)
 		(unit 1)
 		(exclude_from_sim no)
@@
 		(dnp no)
 		(fields_autoplaced yes)
-		(property "Reference" "#PWR036"
-			(at 62.23 44.45 0)
+		(property "Reference" "#PWR02"
+			(at 26.67 43.18 0)
 			(effects
 				(font
@@
 		)
 		(property "Value" "GND"
-			(at 62.23 43.18 0)
+			(at 26.67 41.91 0)
 			(effects
 				(font
@@
 		)
 		(property "Footprint" ""
-			(at 62.23 38.1 0)
+			(at 26.67 36.83 0)
 			(effects
 				(font
@@
 		)
 		(property "Datasheet" ""
-			(at 62.23 38.1 0)
+			(at 26.67 36.83 0)
 			(effects
 				(font
@@
 		)
 		(property "Description" "Power symbol creates a global label with name \"GND\" , ground"
-			(at 62.23 38.1 0)
+			(at 26.67 36.83 0)
 			(effects
 				(font
@@
 			(project "minisumo_pcb"
 				(path "/7b99a4ad-c15f-48f5-acdf-b2b295c8ee3b/d44754c4-1248-482d-a92b-4192f4f09fb1"
-					(reference "#PWR036")
+					(reference "#PWR02")
 					(unit 1)
 				)
