File: Warsztaty/minisumo/minisumo_pcb/programming_connector.kicad_sch (KiCad schematic)
At the start: 1 part

Commit message: koncowy projekt plytki i chyba model tez
Parts:
- renumbered SPI1 to Prog_Con1
Changed lines of the file:
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@@
 		(on_board yes)
 		(dnp no)
-		(property "Reference" "SPI1"
+		(property "Reference" "Prog_Con1"
 			(at 46.99 26.416 0)
 			(effects
@@
 			(project "minisumo_pcb"
 				(path "/7b99a4ad-c15f-48f5-acdf-b2b295c8ee3b/d44754c4-1248-482d-a92b-4192f4f09fb1"
-					(reference "SPI1")
+					(reference "Prog_Con1")
 					(unit 1)
 				)
