File: Warsztaty/minisumo/minisumo_pcb/cnoverter.kicad_sch (KiCad schematic)
At the start: 5 parts, among them Q2 2N7002

Commit message: chyba gotowy schemat
Parts:
- D1: footprint (none) -> LED_THT:LED_D3.0mm
- R1, R2, R3: footprint (none) -> Resistor_SMD:R_0805_2012Metric_Pad1.20x1.40mm_HandSolder
Changed lines of the file:
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@@
 			)
 		)
-		(property "Footprint" ""
+		(property "Footprint" "Resistor_SMD:R_0805_2012Metric_Pad1.20x1.40mm_HandSolder"
 			(at 46.99 41.91 0)
 			(effects
@@
 			)
 		)
-		(property "Footprint" ""
+		(property "Footprint" "Resistor_SMD:R_0805_2012Metric_Pad1.20x1.40mm_HandSolder"
 			(at 33.02 41.91 0)
 			(effects
@@
 			)
 		)
-		(property "Footprint" ""
+		(property "Footprint" "LED_THT:LED_D3.0mm"
 			(at 64.77 38.1 0)
 			(effects
@@
 			)
 		)
-		(property "Footprint" ""
+		(property "Footprint" "Resistor_SMD:R_0805_2012Metric_Pad1.20x1.40mm_HandSolder"
 			(at 64.77 48.26 0)
 			(effects

Commit message: chyba gotowy schemat
Parts:
- renumbered D1 to D5, Q2 to Q4, R3 to R33, R2 to R34, R1 to R35
Connections:
- net MRX: now also Q4.2 (S), R35.2; no longer Q4.3 (D), R33.2
- net STX: now also Q4.3 (D), R33.2; no longer Q4.2 (S), R35.2
