File: Warsztaty/minisumo/minisumo_pcb/motor_driver2.kicad_sch (KiCad schematic)
At the start: 6 parts, among them U2 TB6612FNG

Commit message: chyba gotowy schemat
Parts:
- removed M1: ~, Motors_KoNaR:KoNaR_Motor, symbol Motors_KoNaR:Motor
- C4, C5: footprint Capacitor_Tantalum_SMD:CP_EIA-3528-12_Kemet-T -> Capacitor_SMD:C_0805_2012Metric_Pad1.18x1.45mm_HandSolder
Connections:
- net DIRA_1 renamed DIR1
- net DIRB_1 renamed DIR2
- no-connect marks 0 -> 2
Other:
- note added: "MOTOR_1"
Changed lines of the file:
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@@
-	)
-	(junction
-		(at 72.39 45.72)
-		(diameter 0)
-		(color 0 0 0 0)
 	)
 	(junction
@@
 	)
 	(junction
-		(at 74.93 55.88)
+		(at 72.39 49.53)
 		(diameter 0)
 		(color 0 0 0 0)
@@
 	)
 	(junction
+		(at 74.93 54.61)
+		(diameter 0)
+		(color 0 0 0 0)
+	)
+	(junction
 		(at 77.47 33.02)
 		(diameter 0)
@@
 		(color 0 0 0 0)
 	)
+	(no_connect
+		(at 78.74 49.53)
+	)
+	(no_connect
+		(at 78.74 54.61)
+	)
 	(wire
 		(pts
@@
 	(wire
 		(pts
-			(xy 72.39 38.1) (xy 72.39 45.72)
-		)
-		(stroke
-			(width 0)
-			(type default)
-		)
-	)
-	(wire
-		(pts
 			(xy 30.48 53.34) (xy 30.48 58.42)
 		)
@@
 	(wire
 		(pts
-			(xy 74.93 43.18) (xy 74.93 55.88)
+			(xy 74.93 55.88) (xy 74.93 54.61)
 		)
 		(stroke
@@
 	(wire
 		(pts
-			(xy 72.39 45.72) (xy 83.82 45.72)
+			(xy 74.93 43.18) (xy 74.93 54.61)
 		)
 		(stroke
@@
 	(wire
 		(pts
+			(xy 72.39 49.53) (xy 78.74 49.53)
+		)
+		(stroke
+			(width 0)
+			(type default)
+		)
+	)
+	(wire
+		(pts
 			(xy 72.39 50.8) (xy 68.58 50.8)
 		)
@@
 	(wire
 		(pts
+			(xy 74.93 54.61) (xy 78.74 54.61)
+		)
+		(stroke
+			(width 0)
+			(type default)
+		)
+	)
+	(wire
+		(pts
 			(xy 31.75 25.4) (xy 31.75 27.94)
 		)
@@
 	(wire
 		(pts
+			(xy 72.39 50.8) (xy 72.39 49.53)
+		)
+		(stroke
+			(width 0)
+			(type default)
+		)
+	)
+	(wire
+		(pts
 			(xy 33.02 55.88) (xy 38.1 55.88)
 		)
@@
 	(wire
 		(pts
-			(xy 72.39 45.72) (xy 72.39 50.8)
-		)
-		(stroke
-			(width 0)
-			(type default)
-		)
-	)
-	(wire
-		(pts
 			(xy 45.72 20.32) (xy 45.72 22.86)
 		)
@@
 	(wire
 		(pts
-			(xy 74.93 55.88) (xy 83.82 55.88)
+			(xy 72.39 38.1) (xy 72.39 49.53)
 		)
 		(stroke
@@
 			(font
 				(size 1.27 1.27)
+			)
+		)
+	)
+	(text "MOTOR_1\n\n"
+		(exclude_from_sim no)
+		(at 79.502 53.594 0)
+		(effects
+			(font
+				(size 1.27 1.27)
+				(thickness 0.254)
+				(bold yes)
+				(color 9 191 3 1)
 			)
 		)
@@
 		)
 	)
-	(hierarchical_label "DIRA_1"
+	(hierarchical_label "DIR1"
 		(shape input)
 		(at 29.21 50.8 180)
@@
 		)
 	)
-	(hierarchical_label "DIRB_1"
+	(hierarchical_label "DIR2"
 		(shape input)
 		(at 29.21 58.42 180)
@@
 				(path "/7b99a4ad-c15f-48f5-acdf-b2b295c8ee3b/6ae141c6-db4a-4bb1-a0f3-35ba0e4d6945"
 					(reference "#PWR010")
+					(unit 1)
+				)
+				(path "/7b99a4ad-c15f-48f5-acdf-b2b295c8ee3b/6370311e-bb6b-4c97-a800-647b77b0b74c"
+					(reference "#PWR044")
 					(unit 1)
 				)
@@
 					(unit 1)
 				)
+				(path "/7b99a4ad-c15f-48f5-acdf-b2b295c8ee3b/6370311e-bb6b-4c97-a800-647b77b0b74c"
+					(reference "U13")
+					(unit 1)
+				)
 			)
 		)
@@
 				(path "/7b99a4ad-c15f-48f5-acdf-b2b295c8ee3b/6ae141c6-db4a-4bb1-a0f3-35ba0e4d6945"
 					(reference "#PWR01")
+					(unit 1)
+				)
+				(path "/7b99a4ad-c15f-48f5-acdf-b2b295c8ee3b/6370311e-bb6b-4c97-a800-647b77b0b74c"
+					(reference "#PWR042")
 					(unit 1)
 				)
@@
 					(unit 1)
 				)
+				(path "/7b99a4ad-c15f-48f5-acdf-b2b295c8ee3b/6370311e-bb6b-4c97-a800-647b77b0b74c"
+					(reference "#PWR043")
+					(unit 1)
+				)
 			)
 		)
@@
 					(unit 1)
 				)
+				(path "/7b99a4ad-c15f-48f5-acdf-b2b295c8ee3b/6370311e-bb6b-4c97-a800-647b77b0b74c"
+					(reference "C19")
+					(unit 1)
+				)
 			)
 		)
@@
 			)
 		)
-		(property "Footprint" "Capacitor_Tantalum_SMD:CP_EIA-3528-12_Kemet-T"
+		(property "Footprint" "Capacitor_SMD:C_0805_2012Metric_Pad1.18x1.45mm_HandSolder"
 			(at 26.67 30.48 0)
 			(effects
@@
 					(unit 1)
 				)
-			)
-		)
-	)
-	(symbol
-		(lib_id "Motors_KoNaR:Motor")
-		(at 83.82 50.8 90)
-		(unit 1)
-		(exclude_from_sim no)
-		(in_bom yes)
-		(on_board yes)
-		(dnp no)
-		(fields_autoplaced yes)
-		(property "Reference" "M1"
-			(at 87.63 50.1649 90)
-			(effects
-				(font
-					(size 1.27 1.27)
-				)
-				(justify right)
-			)
-		)
-		(property "Value" "~"
-			(at 87.63 52.07 90)
-			(effects
-				(font
-					(size 1.27 1.27)
-				)
-				(justify right)
-			)
-		)
-		(property "Footprint" "Motors_KoNaR:KoNaR_Motor"
-			(at 87.884 50.8 0)
-			(effects
-				(font
-					(size 1.27 1.27)
-				)
-				(hide yes)
-			)
-		)
-		(property "Datasheet" ""
-			(at 83.82 50.8 0)
-			(effects
-				(font
-					(size 1.27 1.27)
-				)
-				(hide yes)
-			)
-		)
-		(property "Description" ""
-			(at 83.82 50.8 0)
-			(effects
-				(font
-					(size 1.27 1.27)
-				)
-				(hide yes)
-			)
-		)
-		(pin "1"
-		)
-		(pin "2"
-		)
-		(instances
-			(project "minisumo_pcb"
-				(path "/7b99a4ad-c15f-48f5-acdf-b2b295c8ee3b/6ae141c6-db4a-4bb1-a0f3-35ba0e4d6945"
-					(reference "M1")
+				(path "/7b99a4ad-c15f-48f5-acdf-b2b295c8ee3b/6370311e-bb6b-4c97-a800-647b77b0b74c"
+					(reference "C18")
 					(unit 1)
 				)
@@
 				(path "/7b99a4ad-c15f-48f5-acdf-b2b295c8ee3b/6ae141c6-db4a-4bb1-a0f3-35ba0e4d6945"
 					(reference "#PWR012")
+					(unit 1)
+				)
+				(path "/7b99a4ad-c15f-48f5-acdf-b2b295c8ee3b/6370311e-bb6b-4c97-a800-647b77b0b74c"
+					(reference "#PWR040")
 					(unit 1)
 				)
@@
 					(unit 1)
 				)
+				(path "/7b99a4ad-c15f-48f5-acdf-b2b295c8ee3b/6370311e-bb6b-4c97-a800-647b77b0b74c"
+					(reference "#PWR041")
+					(unit 1)
+				)
 			)
 		)
@@
 				(path "/7b99a4ad-c15f-48f5-acdf-b2b295c8ee3b/6ae141c6-db4a-4bb1-a0f3-35ba0e4d6945"
 					(reference "C3")
+					(unit 1)
+				)
+				(path "/7b99a4ad-c15f-48f5-acdf-b2b295c8ee3b/6370311e-bb6b-4c97-a800-647b77b0b74c"
+					(reference "C20")
 					(unit 1)
 				)
@@
 					(unit 1)
 				)
+				(path "/7b99a4ad-c15f-48f5-acdf-b2b295c8ee3b/6370311e-bb6b-4c97-a800-647b77b0b74c"
+					(reference "#PWR051")
+					(unit 1)
+				)
 			)
 		)
@@
 			)
 		)
-		(property "Footprint" "Capacitor_Tantalum_SMD:CP_EIA-3528-12_Kemet-T"
+		(property "Footprint" "Capacitor_SMD:C_0805_2012Metric_Pad1.18x1.45mm_HandSolder"
 			(at 77.47 29.21 0)
 			(effects
@@
 					(unit 1)
 				)
+				(path "/7b99a4ad-c15f-48f5-acdf-b2b295c8ee3b/6370311e-bb6b-4c97-a800-647b77b0b74c"
+					(reference "C23")
+					(unit 1)
+				)
