File: Warsztaty/minisumo/minisumo_pcb/inverter.kicad_sch (KiCad schematic)
At the start: 2 parts, among them U1 SN74LVC2G14DBV

Commit message: chyba gotowy schemat
Parts:
- C7: footprint (none) -> Capacitor_SMD:C_0805_2012Metric_Pad1.18x1.45mm_HandSolder
Changed lines of the file:
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@@
 			)
 		)
-		(property "Footprint" ""
+		(property "Footprint" "Capacitor_SMD:C_0805_2012Metric_Pad1.18x1.45mm_HandSolder"
 			(at 63.5 38.1 0)
 			(effects

Commit message: chyba gotowy schemat
Connections:
- net DIR1_1 renamed DIRA_2
- net DIR1_2 renamed DIRB_2
- net DIR2_1 renamed DIRA_1
- net DIR2_2 renamed DIRB_1
Changed lines of the file:
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@@
 		)
 	)
-	(hierarchical_label "DIR1_1"
+	(hierarchical_label "DIRA_1"
+		(shape input)
+		(at 49.53 35.56 0)
+		(fields_autoplaced yes)
+		(effects
+			(font
+				(size 0.762 0.762)
+			)
+			(justify left)
+		)
+	)
+	(hierarchical_label "DIRB_1"
+		(shape input)
+		(at 29.21 35.56 180)
+		(fields_autoplaced yes)
+		(effects
+			(font
+				(size 0.762 0.762)
+			)
+			(justify right)
+		)
+	)
+	(hierarchical_label "DIRB_2"
+		(shape input)
+		(at 29.21 40.64 180)
+		(fields_autoplaced yes)
+		(effects
+			(font
+				(size 0.762 0.762)
+			)
+			(justify right)
+		)
+	)
+	(hierarchical_label "DIRA_2"
 		(shape input)
 		(at 49.53 40.64 0)
@@
 		)
 	)
-	(hierarchical_label "DIR2_1"
-		(shape input)
-		(at 49.53 35.56 0)
-		(fields_autoplaced yes)
-		(effects
-			(font
-				(size 0.762 0.762)
-			)
-			(justify left)
-		)
-	)
-	(hierarchical_label "DIR2_2"
-		(shape input)
-		(at 29.21 35.56 180)
-		(fields_autoplaced yes)
-		(effects
-			(font
-				(size 0.762 0.762)
-			)
-			(justify right)
-		)
-	)
-	(hierarchical_label "DIR1_2"
-		(shape input)
-		(at 29.21 40.64 180)
-		(fields_autoplaced yes)
-		(effects
-			(font
-				(size 0.762 0.762)
-			)
-			(justify right)
-		)
-	)

Commit message: stan przed usunięciem jednego czujnika lini
Parts:
- C7: footprint Capacitor_SMD:C_0805_2012Metric_Pad1.18x1.45mm_HandSolder -> Capacitor_SMD:C_0805_2012Metric
Changed lines of the file:
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@@
 			)
 		)
-		(property "Footprint" "Capacitor_SMD:C_0805_2012Metric_Pad1.18x1.45mm_HandSolder"
+		(property "Footprint" "Capacitor_SMD:C_0805_2012Metric"
 			(at 63.5 38.1 0)
 			(effects

Commit message: koncowy projekt plytki i chyba model tez
Parts:
- renumbered U1 to INVERTER1
Changed lines of the file:
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@@
 		(dnp no)
 		(fields_autoplaced yes)
-		(property "Reference" "U1"
+		(property "Reference" "INVERTER1"
 			(at 41.5641 25.4 0)
 			(effects
@@
 			(project "minisumo_pcb"
 				(path "/7b99a4ad-c15f-48f5-acdf-b2b295c8ee3b/b8d919d3-78c3-4a57-ab4a-a567d8eddd6d"
-					(reference "U1")
+					(reference "INVERTER1")
 					(unit 1)
 				)
