File: Warsztaty/minisumo/minisumo_pcb/minisumo_pcb.kicad_sch (KiCad schematic)
At the start: 0 parts

Commit message: chyba gotowy schemat
Other:
- removed sheet converter_GPIO1_1
- removed sheet converter_GPIO1_2
- removed sheet converter_GPIO1_4
- removed sheet converter_SCL
- removed sheet converter_SDA
- removed sheet converter_XSHUT_1
- removed sheet converter_XSHUT_2
- removed sheet converter_XSHUT_3
- removed sheet converter_XSHUT_4
- sheet inverter ports: added DIRA_1, DIRA_2, DIRB_1, DIRB_2; removed DIR1_1, DIR1_2, DIR2_1, DIR2_2
- sheet motor_driver1 ports: added DIRA_1, DIRB_1; removed DIR1_1, DIR2_1
- sheet motor_driver2: file motor_driver1.kicad_sch -> motor_driver2_sch.kicad_sch
- sheet motor_driver2 ports: added DIRA_2, DIRB_2; removed DIR1_2, DIR2_2
- sheet sensor1 ports: added G1, X1; removed GPIO1_1, XSHUT_1
- sheet sensor2: file sensor1.kicad_sch -> sensor2.kicad_sch
- sheet sensor2 ports: added G2, X2; removed GPIO1_1, XSHUT_1
- sheet sensor3: file sensor1.kicad_sch -> sensor3.kicad_sch
- sheet sensor3 ports: added G3, X3; removed GPIO1_1, XSHUT_1
- sheet sensor4: file sensor1.kicad_sch -> sensor4.kicad_sch
- sheet sensor4 ports: added G4, X4; removed GPIO1_1, XSHUT_1
- sheet uC ports: added DIRB_1, DIRB_2; removed DIR1_2, DIR2_2, XTAL1, XTAL2

Commit message: Wstępny wyglad robota i płytki
Other:
- sheet uC ports: added STARTER; removed none
Changed lines of the file:
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@@
+	(wire
+		(pts
+			(xy 172.72 142.24) (xy 176.53 142.24)
+		)
+		(stroke
+			(width 0)
+			(type default)
+		)
+	)
 	(wire
 		(pts
@@
 		(pts
 			(xy 105.41 81.28) (xy 113.03 81.28)
-		)
-		(stroke
-			(width 0)
-			(type default)
-		)
-	)
-	(wire
-		(pts
-			(xy 172.72 142.24) (xy 176.53 142.24)
 		)
 		(stroke
@@
 			)
 		)
+		(pin "LS1" input
+			(at 172.72 137.16 0)
+			(effects
+				(font
+					(size 1.27 1.27)
+				)
+				(justify right)
+			)
+		)
+		(pin "LS2" input
+			(at 172.72 139.7 0)
+			(effects
+				(font
+					(size 1.27 1.27)
+				)
+				(justify right)
+			)
+		)
+		(pin "RST" input
+			(at 172.72 69.85 0)
+			(effects
+				(font
+					(size 1.27 1.27)
+				)
+				(justify right)
+			)
+		)
+		(pin "SCK" input
+			(at 172.72 72.39 0)
+			(effects
+				(font
+					(size 1.27 1.27)
+				)
+				(justify right)
+			)
+		)
+		(pin "XSHUT_4" input
+			(at 134.62 99.06 180)
+			(effects
+				(font
+					(size 1.27 1.27)
+				)
+				(justify left)
+			)
+		)
+		(pin "XSHUT_3" input
+			(at 134.62 91.44 180)
+			(effects
+				(font
+					(size 1.27 1.27)
+				)
+				(justify left)
+			)
+		)
+		(pin "XSHUT_2" input
+			(at 134.62 83.82 180)
+			(effects
+				(font
+					(size 1.27 1.27)
+				)
+				(justify left)
+			)
+		)
+		(pin "XSHUT_1" input
+			(at 134.62 76.2 180)
+			(effects
+				(font
+					(size 1.27 1.27)
+				)
+				(justify left)
+			)
+		)
+		(pin "DIRB_2" input
+			(at 172.72 96.52 0)
+			(effects
+				(font
+					(size 1.27 1.27)
+				)
+				(justify right)
+			)
+		)
+		(pin "DIRB_1" input
+			(at 172.72 92.71 0)
+			(effects
+				(font
+					(size 1.27 1.27)
+				)
+				(justify right)
+			)
+		)
+		(pin "STARTER" input
+			(at 172.72 115.57 0)
+			(effects
+				(font
+					(size 1.27 1.27)
+				)
+				(justify right)
+			)
+		)
 		(pin "LS3" input
 			(at 172.72 142.24 0)
-			(effects
-				(font
-					(size 1.27 1.27)
-				)
-				(justify right)
-			)
-		)
-		(pin "LS1" input
-			(at 172.72 137.16 0)
-			(effects
-				(font
-					(size 1.27 1.27)
-				)
-				(justify right)
-			)
-		)
-		(pin "LS2" input
-			(at 172.72 139.7 0)
-			(effects
-				(font
-					(size 1.27 1.27)
-				)
-				(justify right)
-			)
-		)
-		(pin "RST" input
-			(at 172.72 69.85 0)
-			(effects
-				(font
-					(size 1.27 1.27)
-				)
-				(justify right)
-			)
-		)
-		(pin "SCK" input
-			(at 172.72 72.39 0)
-			(effects
-				(font
-					(size 1.27 1.27)
-				)
-				(justify right)
-			)
-		)
-		(pin "XSHUT_4" input
-			(at 134.62 99.06 180)
-			(effects
-				(font
-					(size 1.27 1.27)
-				)
-				(justify left)
-			)
-		)
-		(pin "XSHUT_3" input
-			(at 134.62 91.44 180)
-			(effects
-				(font
-					(size 1.27 1.27)
-				)
-				(justify left)
-			)
-		)
-		(pin "XSHUT_2" input
-			(at 134.62 83.82 180)
-			(effects
-				(font
-					(size 1.27 1.27)
-				)
-				(justify left)
-			)
-		)
-		(pin "XSHUT_1" input
-			(at 134.62 76.2 180)
-			(effects
-				(font
-					(size 1.27 1.27)
-				)
-				(justify left)
-			)
-		)
-		(pin "DIRB_2" input
-			(at 172.72 96.52 0)
-			(effects
-				(font
-					(size 1.27 1.27)
-				)
-				(justify right)
-			)
-		)
-		(pin "DIRB_1" input
-			(at 172.72 92.71 0)
 			(effects
 				(font
@@
 		)
 		(pin "LS2" input
-			(at 176.53 142.24 180)
-			(effects
-				(font
-					(size 1.27 1.27)
-				)
-				(justify left)
-			)
-		)
-		(pin "LS3" input
 			(at 176.53 139.7 180)
 			(effects
@@
 			(effects
 				(font
+					(size 1.27 1.27)
+				)
+				(justify left)
+			)
+		)
+		(pin "LS3" output
+			(at 176.53 142.24 180)
+			(effects
+				(font

Commit message: prawdopodobnie koncowa wersja płytki
Other:
- sheet sensor1 ports: added XSHUT_1; removed X1
- sheet sensor2 ports: added XSHUT_2; removed X2
- sheet sensor3 ports: added XSHUT_3; removed X3
- sheet sensor4 ports: added XSHUT_4; removed X4
Changed lines of the file:
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@@
-			)
-		)
-		(pin "X2" input
-			(at 105.41 86.36 0)
-			(effects
-				(font
-					(size 1.27 1.27)
-				)
-				(justify right)
 			)
 		)
@@
 			)
 		)
+		(pin "XSHUT_2" input
+			(at 105.41 86.36 0)
+			(effects
+				(font
+					(size 1.27 1.27)
+				)
+				(justify right)
+			)
+		)
 		(instances
 			(project "minisumo_pcb"
@@
 			)
 		)
-		(pin "X1" input
-			(at 105.41 67.31 0)
-			(effects
-				(font
-					(size 1.27 1.27)
-				)
-				(justify right)
-			)
-		)
 		(pin "SDA" input
 			(at 105.41 64.77 0)
@@
 			)
 		)
+		(pin "XSHUT_1" input
+			(at 105.41 67.31 0)
+			(effects
+				(font
+					(size 1.27 1.27)
+				)
+				(justify right)
+			)
+		)
 		(instances
 			(project "minisumo_pcb"
@@
 			)
 		)
-		(pin "X3" input
-			(at 105.41 104.14 0)
-			(effects
-				(font
-					(size 1.27 1.27)
-				)
-				(justify right)
-			)
-		)
 		(pin "SDA" input
 			(at 105.41 101.6 0)
@@
 			)
 		)
+		(pin "XSHUT_3" input
+			(at 105.41 104.14 0)
+			(effects
+				(font
+					(size 1.27 1.27)
+				)
+				(justify right)
+			)
+		)
 		(instances
 			(project "minisumo_pcb"
@@
 			)
 		)
-		(pin "X4" input
-			(at 105.41 123.19 0)
-			(effects
-				(font
-					(size 1.27 1.27)
-				)
-				(justify right)
-			)
-		)
 		(pin "SCL" input
 			(at 105.41 118.11 0)
 			(effects
 				(font
+					(size 1.27 1.27)
+				)
+				(justify right)
+			)
+		)
+		(pin "XSHUT_4" input
+			(at 105.41 123.19 0)
+			(effects
+				(font
