File: Warsztaty/minisumo/minisumo_pcb/sensor3.kicad_sch (KiCad schematic)
At the start: 1 part

Commit message: chyba gotowy schemat
Parts:
- removed SPI1: MTSW-103-23-F-D-230, MTSW-103-23-F-D-230:SAMTEC_MTSW-103-23-F-D-230, symbol MTSW-103-23-F-D-230:MTSW-103-23-F-D-230
- added SPI4: MTSW-103-23-F-D-230, MTSW-103-23-F-D-230:SAMTEC_MTSW-103-23-F-D-230, symbol MTSW-103-23-F-D-230:MTSW-103-23-F-D-230
Connections:
- net +5V: now also SPI4.02
- net GND: now also SPI4.01
- new net G3: SPI4.06
- new net SCL: SPI4.04
- new net SDA: SPI4.03
- new net X3: SPI4.05
Other:
- note added: "Sensor3"
- note removed: "Programming connector"
Changed lines of the file:
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@@
 	(wire
 		(pts
-			(xy 62.23 35.56) (xy 62.23 39.37)
-		)
-		(stroke
-			(width 0)
-			(type default)
-		)
-	)
-	(wire
-		(pts
-			(xy 59.69 35.56) (xy 62.23 35.56)
+			(xy 59.69 33.02) (xy 60.96 33.02)
 		)
 		(stroke
@@
 	(wire
 		(pts
+			(xy 24.13 38.1) (xy 24.13 30.48)
+		)
+		(stroke
+			(width 0)
+			(type default)
+		)
+	)
+	(wire
+		(pts
+			(xy 59.69 35.56) (xy 60.96 35.56)
+		)
+		(stroke
+			(width 0)
+			(type default)
+		)
+	)
+	(wire
+		(pts
+			(xy 33.02 33.02) (xy 34.29 33.02)
+		)
+		(stroke
+			(width 0)
+			(type default)
+		)
+	)
+	(wire
+		(pts
+			(xy 24.13 30.48) (xy 34.29 30.48)
+		)
+		(stroke
+			(width 0)
+			(type default)
+		)
+	)
+	(wire
+		(pts
 			(xy 62.23 29.21) (xy 62.23 30.48)
 		)
@@
 	(wire
 		(pts
-			(xy 33.02 33.02) (xy 34.29 33.02)
-		)
-		(stroke
-			(width 0)
-			(type default)
-		)
-	)
-	(wire
-		(pts
 			(xy 59.69 30.48) (xy 62.23 30.48)
-		)
-		(stroke
-			(width 0)
-			(type default)
-		)
-	)
-	(wire
-		(pts
-			(xy 59.69 33.02) (xy 60.96 33.02)
 		)
 		(stroke
@@
 		)
 	)
-	(text "Programming connector"
+	(text "Sensor3\n\n"
 		(exclude_from_sim no)
 		(at 27.686 16.256 0)
@@
 		)
 	)
-	(hierarchical_label "SCK"
+	(hierarchical_label "X3"
 		(shape input)
-		(at 33.02 33.02 180)
+		(at 33.02 35.56 180)
 		(fields_autoplaced yes)
 		(effects
@@
 		)
 	)
-	(hierarchical_label "RST"
+	(hierarchical_label "G3"
 		(shape input)
-		(at 33.02 35.56 180)
+		(at 60.96 35.56 0)
 		(fields_autoplaced yes)
 		(effects
@@
 				(size 0.762 0.762)
 			)
-			(justify right)
-		)
-	)
-	(hierarchical_label "MOSI"
+			(justify left)
+		)
+	)
+	(hierarchical_label "SCL"
 		(shape input)
 		(at 60.96 33.02 0)
@@
 		)
 	)
-	(hierarchical_label "MISO"
+	(hierarchical_label "SDA"
 		(shape input)
-		(at 34.29 30.48 180)
+		(at 33.02 33.02 180)
 		(fields_autoplaced yes)
 		(effects
@@
 			)
 			(justify right)
+		)
+	)
+	(symbol
+		(lib_id "power:GND")
+		(at 24.13 38.1 0)
+		(unit 1)
+		(exclude_from_sim no)
+		(in_bom yes)
+		(on_board yes)
+		(dnp no)
+		(fields_autoplaced yes)
+		(property "Reference" "#PWR017"
+			(at 24.13 44.45 0)
+			(effects
+				(font
+					(size 1.27 1.27)
+				)
+				(hide yes)
+			)
+		)
+		(property "Value" "GND"
+			(at 24.13 43.18 0)
+			(effects
+				(font
+					(size 1.27 1.27)
+				)
+			)
+		)
+		(property "Footprint" ""
+			(at 24.13 38.1 0)
+			(effects
+				(font
+					(size 1.27 1.27)
+				)
+				(hide yes)
+			)
+		)
+		(property "Datasheet" ""
+			(at 24.13 38.1 0)
+			(effects
+				(font
+					(size 1.27 1.27)
+				)
+				(hide yes)
+			)
+		)
+		(property "Description" "Power symbol creates a global label with name \"GND\" , ground"
+			(at 24.13 38.1 0)
+			(effects
+				(font
+					(size 1.27 1.27)
+				)
+				(hide yes)
+			)
+		)
+		(pin "1"
+		)
+		(instances
+			(project "minisumo_pcb"
+				(path "/7b99a4ad-c15f-48f5-acdf-b2b295c8ee3b/b1e52e37-65e3-4b7a-ac18-46ca748af580"
+					(reference "#PWR017")
+					(unit 1)
+				)
+			)
+		)
+	)
+	(symbol
+		(lib_id "power:+5V")
+		(at 62.23 29.21 0)
+		(unit 1)
+		(exclude_from_sim no)
+		(in_bom yes)
+		(on_board yes)
+		(dnp no)
+		(fields_autoplaced yes)
+		(property "Reference" "#PWR020"
+			(at 62.23 33.02 0)
+			(effects
+				(font
+					(size 1.27 1.27)
+				)
+				(hide yes)
+			)
+		)
+		(property "Value" "+5V"
+			(at 62.23 24.13 0)
+			(effects
+				(font
+					(size 1.27 1.27)
+				)
+			)
+		)
+		(property "Footprint" ""
+			(at 62.23 29.21 0)
+			(effects
+				(font
+					(size 1.27 1.27)
+				)
+				(hide yes)
+			)
+		)
+		(property "Datasheet" ""
+			(at 62.23 29.21 0)
+			(effects
+				(font
+					(size 1.27 1.27)
+				)
+				(hide yes)
+			)
+		)
+		(property "Description" "Power symbol creates a global label with name \"+5V\""
+			(at 62.23 29.21 0)
+			(effects
+				(font
+					(size 1.27 1.27)
+				)
+				(hide yes)
+			)
+		)
+		(pin "1"
+		)
+		(instances
+			(project "minisumo_pcb"
+				(path "/7b99a4ad-c15f-48f5-acdf-b2b295c8ee3b/b1e52e37-65e3-4b7a-ac18-46ca748af580"
+					(reference "#PWR020")
+					(unit 1)
+				)
+			)
 		)
 	)
@@
 		(on_board yes)
 		(dnp no)
-		(property "Reference" "SPI1"
+		(property "Reference" "SPI4"
 			(at 46.99 26.416 0)
 			(effects
@@
 		(instances
 			(project "minisumo_pcb"
-				(path "/7b99a4ad-c15f-48f5-acdf-b2b295c8ee3b/d44754c4-1248-482d-a92b-4192f4f09fb1"
-					(reference "SPI1")
+				(path "/7b99a4ad-c15f-48f5-acdf-b2b295c8ee3b/b1e52e37-65e3-4b7a-ac18-46ca748af580"
+					(reference "SPI4")
 					(unit 1)
 				)
-			)
-		)
-	)
-	(symbol
-		(lib_id "power:GND")
-		(at 62.23 39.37 0)
-		(unit 1)
-		(exclude_from_sim no)
-		(in_bom yes)
-		(on_board yes)
-		(dnp no)
-		(fields_autoplaced yes)
-		(property "Reference" "#PWR02"
-			(at 62.23 45.72 0)
-			(effects
-				(font
-					(size 1.27 1.27)
-				)
-				(hide yes)
-			)
-		)
-		(property "Value" "GND"
-			(at 62.23 44.45 0)
-			(effects
-				(font
-					(size 1.27 1.27)
-				)
-			)
-		)
-		(property "Footprint" ""
-			(at 62.23 39.37 0)
-			(effects
-				(font
-					(size 1.27 1.27)
-				)
-				(hide yes)
-			)
-		)
-		(property "Datasheet" ""
-			(at 62.23 39.37 0)
-			(effects
-				(font
-					(size 1.27 1.27)
-				)
-				(hide yes)
-			)
-		)
-		(property "Description" "Power symbol creates a global label with name \"GND\" , ground"
-			(at 62.23 39.37 0)
-			(effects
-				(font
-					(size 1.27 1.27)
-				)
-				(hide yes)
-			)
-		)
-		(pin "1"
-		)
-		(instances
-			(project "minisumo_pcb"
-				(path "/7b99a4ad-c15f-48f5-acdf-b2b295c8ee3b/d44754c4-1248-482d-a92b-4192f4f09fb1"
-					(reference "#PWR02")
-					(unit 1)
-				)
-			)
-		)
-	)
-	(symbol
-		(lib_id "power:+5V")
-		(at 62.23 29.21 0)
-		(unit 1)
-		(exclude_from_sim no)
-		(in_bom yes)
-		(on_board yes)
-		(dnp no)
-		(fields_autoplaced yes)
-		(property "Reference" "#PWR035"
-			(at 62.23 33.02 0)
-			(effects
-				(font
-					(size 1.27 1.27)
-				)
-				(hide yes)
-			)
-		)
-		(property "Value" "+5V"
-			(at 62.23 24.13 0)
-			(effects
-				(font
-					(size 1.27 1.27)
-				)
-			)
-		)
-		(property "Footprint" ""
-			(at 62.23 29.21 0)
-			(effects
-				(font
-					(size 1.27 1.27)
-				)
-				(hide yes)
-			)
-		)
-		(property "Datasheet" ""
-			(at 62.23 29.21 0)
-			(effects
-				(font
-					(size 1.27 1.27)
-				)
-				(hide yes)
-			)
-		)
-		(property "Description" "Power symbol creates a global label with name \"+5V\""
-			(at 62.23 29.21 0)
-			(effects
-				(font
-					(size 1.27 1.27)
-				)
-				(hide yes)
-			)
-		)
-		(pin "1"
-		)
-		(instances
-			(project "minisumo_pcb"
-				(path "/7b99a4ad-c15f-48f5-acdf-b2b295c8ee3b/d44754c4-1248-482d-a92b-4192f4f09fb1"
-					(reference "#PWR035")
-					(unit 1)
-				)

Commit message: stan przed usunięciem jednego czujnika lini
Parts:
- added R10: 10k, Resistor_SMD:R_0805_2012Metric, symbol Device:R_Small
- added R9: 20k, Resistor_SMD:R_0805_2012Metric, symbol Device:R_Small
Connections:
- net GND: now also R9.1
- net X3: now also R10.2, R9.2; no longer SPI4.05
- new net: R10.1, SPI4.05

Commit message: Wstępny wyglad robota i płytki
Connections:
- net X3: no longer R9.2
- net at R10.1, SPI4.05: now also R9.2
Other:
- moved on the sheet: R10, R9
Changed lines of the file:
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@@
 	(paper "A4")
 	(junction
-		(at 24.13 35.56)
+		(at 30.48 35.56)
 		(diameter 0)
 		(color 0 0 0 0)
@@
 	(wire
 		(pts
-			(xy 24.13 35.56) (xy 25.4 35.56)
-		)
-		(stroke
-			(width 0)
-			(type default)
-		)
-	)
-	(wire
-		(pts
 			(xy 59.69 35.56) (xy 60.96 35.56)
 		)
@@
 	(wire
 		(pts
+			(xy 30.48 35.56) (xy 30.48 36.83)
+		)
+		(stroke
+			(width 0)
+			(type default)
+		)
+	)
+	(wire
+		(pts
+			(xy 30.48 35.56) (xy 34.29 35.56)
+		)
+		(stroke
+			(width 0)
+			(type default)
+		)
+	)
+	(wire
+		(pts
 			(xy 33.02 33.02) (xy 34.29 33.02)
 		)
@@
 	(wire
 		(pts
-			(xy 20.32 35.56) (xy 24.13 35.56)
-		)
-		(stroke
-			(width 0)
-			(type default)
-		)
-	)
-	(wire
-		(pts
-			(xy 24.13 41.91) (xy 24.13 44.45)
+			(xy 20.32 35.56) (xy 21.59 35.56)
+		)
+		(stroke
+			(width 0)
+			(type default)
+		)
+	)
+	(wire
+		(pts
+			(xy 30.48 41.91) (xy 30.48 44.45)
 		)
 		(stroke
@@
 	(wire
 		(pts
-			(xy 30.48 35.56) (xy 34.29 35.56)
-		)
-		(stroke
-			(width 0)
-			(type default)
-		)
-	)
-	(wire
-		(pts
-			(xy 24.13 35.56) (xy 24.13 36.83)
+			(xy 26.67 35.56) (xy 30.48 35.56)
 		)
 		(stroke
@@
 	(symbol
 		(lib_id "power:GND")
-		(at 24.13 44.45 0)
+		(at 30.48 44.45 0)
 		(unit 1)
 		(exclude_from_sim no)
@@
 		(dnp no)
 		(property "Reference" "#PWR031"
-			(at 24.13 50.8 0)
+			(at 30.48 50.8 0)
 			(effects
 				(font
@@
 		)
 		(property "Value" "GND"
-			(at 24.13 48.26 0)
+			(at 30.48 48.26 0)
 			(effects
 				(font
@@
 		)
 		(property "Footprint" ""
-			(at 24.13 44.45 0)
+			(at 30.48 44.45 0)
 			(effects
 				(font
@@
 		)
 		(property "Datasheet" ""
-			(at 24.13 44.45 0)
+			(at 30.48 44.45 0)
 			(effects
 				(font
@@
 		)
 		(property "Description" "Power symbol creates a global label with name \"GND\" , ground"
-			(at 24.13 44.45 0)
+			(at 30.48 44.45 0)
 			(effects
 				(font
@@
 	(symbol
 		(lib_id "Device:R_Small")
-		(at 27.94 35.56 270)
+		(at 24.13 35.56 270)
 		(unit 1)
 		(exclude_from_sim no)
@@
 		(dnp no)
 		(property "Reference" "R10"
-			(at 27.94 37.338 90)
+			(at 24.13 37.338 90)
 			(effects
 				(font
@@
 		)
 		(property "Value" "10k"
-			(at 27.94 33.782 90)
+			(at 24.13 33.782 90)
 			(effects
 				(font
@@
 		)
 		(property "Footprint" "Resistor_SMD:R_0805_2012Metric"
-			(at 27.94 35.56 0)
+			(at 24.13 35.56 0)
 			(effects
 				(font
@@
 		)
 		(property "Datasheet" "~"
-			(at 27.94 35.56 0)
+			(at 24.13 35.56 0)
 			(effects
 				(font
@@
 		)
 		(property "Description" "Resistor, small symbol"
-			(at 27.94 35.56 0)
+			(at 24.13 35.56 0)
 			(effects
 				(font
@@
 	(symbol
 		(lib_id "Device:R_Small")
-		(at 24.13 39.37 180)
+		(at 30.48 39.37 180)
 		(unit 1)
 		(exclude_from_sim no)
@@
 		(dnp no)
 		(property "Reference" "R9"
-			(at 22.352 39.37 90)
+			(at 28.702 39.37 90)
 			(effects
 				(font
@@
 		)
 		(property "Value" "20k"
-			(at 25.908 39.37 90)
+			(at 32.258 39.37 90)
 			(effects
 				(font
@@
 		)
 		(property "Footprint" "Resistor_SMD:R_0805_2012Metric"
-			(at 24.13 39.37 0)
+			(at 30.48 39.37 0)
 			(effects
 				(font
@@
 		)
 		(property "Datasheet" "~"
-			(at 24.13 39.37 0)
+			(at 30.48 39.37 0)
 			(effects
 				(font
@@
 		)
 		(property "Description" "Resistor, small symbol"
-			(at 24.13 39.37 0)
-			(effects
-				(font
+			(at 30.48 39.37 0)
+			(effects
+				(font

Commit message: koncowy projekt plytki i chyba model tez
Parts:
- renumbered SPI4 to ES3
Changed lines of the file:
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@@
 		(on_board yes)
 		(dnp no)
-		(property "Reference" "SPI4"
+		(property "Reference" "ES3"
 			(at 46.99 26.416 0)
 			(effects
@@
 			(project "minisumo_pcb"
 				(path "/7b99a4ad-c15f-48f5-acdf-b2b295c8ee3b/b1e52e37-65e3-4b7a-ac18-46ca748af580"
-					(reference "SPI4")
+					(reference "ES3")
 					(unit 1)
 				)

Commit message: prawdopodobnie koncowa wersja płytki
Connections:
- net X3 renamed XSHUT_3
Changed lines of the file:
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@@
 		)
 	)
-	(hierarchical_label "X3"
+	(hierarchical_label "XSHUT_3"
 		(shape input)
 		(at 20.32 35.56 180)
