File: Warsztaty/minisumo/minisumo_pcb/minisumo_pcb.kicad_pcb (KiCad board)
At the start: 2 copper layers, 0 parts

Commit message: chyba gotowy schemat
Parts:
- added B1: SKHLAAA010, SKHLAAA010:SKHLAAA010, F.Cu at (87.1, 87.8)
- added C1: 22p, Capacitor_SMD:C_0805_2012Metric_Pad1.18x1.45mm_HandSolder, F.Cu at (70.2, 69.5)
- added C10: 10u, Capacitor_SMD:C_0805_2012Metric_Pad1.18x1.45mm_HandSolder, F.Cu at (87.9, 45.8)
- added C11: 10uF, Capacitor_SMD:C_0805_2012Metric_Pad1.18x1.45mm_HandSolder, F.Cu at (87.9, 48.8)
- added C12: 10uF, Capacitor_SMD:C_0805_2012Metric_Pad1.18x1.45mm_HandSolder, F.Cu at (87.9, 51.8)
- added C13: 4,7uF, Capacitor_SMD:C_0805_2012Metric_Pad1.18x1.45mm_HandSolder, F.Cu at (225.1, 79.7)
- added C14: 100nF, Capacitor_SMD:C_0805_2012Metric_Pad1.18x1.45mm_HandSolder, F.Cu at (190.4, 104.5)
- added C15: 4,7uF, Capacitor_SMD:C_0805_2012Metric_Pad1.18x1.45mm_HandSolder, F.Cu at (190.4, 107.5)
- added C16: 100nF, Capacitor_SMD:C_0805_2012Metric_Pad1.18x1.45mm_HandSolder, F.Cu at (203.8, 90.7)
- added C17: 4,7uF, Capacitor_SMD:C_0805_2012Metric_Pad1.18x1.45mm_HandSolder, F.Cu at (203.8, 93.8)
- added C18: 10uF, Capacitor_SMD:C_0805_2012Metric_Pad1.18x1.45mm_HandSolder, F.Cu at (185.6, 72.5)
- added C19: 10nF, Capacitor_SMD:C_0805_2012Metric_Pad1.18x1.45mm_HandSolder, F.Cu at (185.6, 75.5)
- added C2: 22p, Capacitor_SMD:C_0805_2012Metric_Pad1.18x1.45mm_HandSolder, F.Cu at (70.2, 72.5)
- added C20: 10nF, Capacitor_SMD:C_0805_2012Metric_Pad1.18x1.45mm_HandSolder, F.Cu at (185.6, 78.5)
- added C21: 100nF, Capacitor_SMD:C_0805_2012Metric_Pad1.18x1.45mm_HandSolder, F.Cu at (190.4, 90.7)
- added C22: 4,7uF, Capacitor_SMD:C_0805_2012Metric_Pad1.18x1.45mm_HandSolder, F.Cu at (190.4, 93.8)
- added C23: 10uF, Capacitor_SMD:C_0805_2012Metric_Pad1.18x1.45mm_HandSolder, F.Cu at (185.6, 81.5)
- added C24: 1uF, Capacitor_SMD:C_0805_2012Metric_Pad1.18x1.45mm_HandSolder, F.Cu at (70.2, 75.5)
- added C25: 100nF, Capacitor_SMD:C_0805_2012Metric_Pad1.18x1.45mm_HandSolder, F.Cu at (70.2, 78.5)
- added C26: 1uF, Capacitor_SMD:C_0805_2012Metric_Pad1.18x1.45mm_HandSolder, F.Cu at (70.2, 81.5)
- added C3: 10nF, Capacitor_SMD:C_0805_2012Metric_Pad1.18x1.45mm_HandSolder, F.Cu at (203.0, 72.5)
- added C4: 10uF, Capacitor_SMD:C_0805_2012Metric_Pad1.18x1.45mm_HandSolder, F.Cu at (203.0, 75.5)
- added C5: 10uF, Capacitor_SMD:C_0805_2012Metric_Pad1.18x1.45mm_HandSolder, F.Cu at (203.0, 78.5)
- added C6: 10nF, Capacitor_SMD:C_0805_2012Metric_Pad1.18x1.45mm_HandSolder, F.Cu at (203.0, 81.5)
- added C7: 100nF, Capacitor_SMD:C_0805_2012Metric_Pad1.18x1.45mm_HandSolder, F.Cu at (226.9, 62.6)
- added C8: 100nF, Capacitor_SMD:C_0805_2012Metric_Pad1.18x1.45mm_HandSolder, F.Cu at (225.1, 76.7)
- added C9: 10u, Capacitor_SMD:C_0805_2012Metric_Pad1.18x1.45mm_HandSolder, F.Cu at (87.9, 42.8)
- added D1: blue, LED_THT:LED_D3.0mm, F.Cu at (218.3, 59.2)
- added D10: blue, LED_THT:LED_D3.0mm, F.Cu at (193.0, 47.1)
- added D11: blue, LED_THT:LED_D3.0mm, F.Cu at (205.6, 47.1)
- added D12: blue, LED_THT:LED_D3.0mm, F.Cu at (205.6, 59.2)
- added D2: red, LED_THT:LED_D3.0mm, F.Cu at (86.5, 76.9)
- added D3: green, LED_THT:LED_D3.0mm, F.Cu at (86.5, 82.5)
- added D4: blue, LED_THT:LED_D3.0mm, F.Cu at (203.0, 101.6)
- added D5: blue, LED_THT:LED_D3.0mm, F.Cu at (193.0, 59.2)
- added D6: blue, LED_THT:LED_D3.0mm, F.Cu at (216.4, 112.1)
- added D7: blue, LED_THT:LED_D3.0mm, F.Cu at (216.4, 100.0)
- added D8: blue, LED_THT:LED_D3.0mm, F.Cu at (218.3, 47.1)
- added D9: blue, LED_THT:LED_D3.0mm, F.Cu at (216.4, 87.8)
- added J1: HTSW-102-08-L-S, HTSW-102-08-L-S:SAMTEC_HTSW-102-08-L-S, F.Cu at (58.7, 120.5)
- added J2: Conn_01x02_Pin, Connector_JST:JST_EH_B2B-EH-A_1x02_P2.50mm_Vertical, F.Cu at (178.5, 59.0)
- added Q1: PMOS, Package_TO_SOT_SMD:SOT-23-3, F.Cu at (88.1, 61.5)
- added Q10: 2N7002, Package_TO_SOT_SMD:SOT-23, F.Cu at (206.4, 52.2)
- added Q11: 2N7002, Package_TO_SOT_SMD:SOT-23, F.Cu at (206.4, 64.4)
- added Q2: 2N7002, Package_TO_SOT_SMD:SOT-23, F.Cu at (219.1, 64.4)
- added Q3: 2N7002, Package_TO_SOT_SMD:SOT-23, F.Cu at (203.8, 106.8)
- added Q4: 2N7002, Package_TO_SOT_SMD:SOT-23, F.Cu at (193.8, 64.4)
- added Q5: 2N7002, Package_TO_SOT_SMD:SOT-23, F.Cu at (217.2, 117.3)
- added Q6: 2N7002, Package_TO_SOT_SMD:SOT-23, F.Cu at (217.2, 105.1)
- added Q7: 2N7002, Package_TO_SOT_SMD:SOT-23, F.Cu at (219.1, 52.2)
- added Q8: 2N7002, Package_TO_SOT_SMD:SOT-23, F.Cu at (217.2, 93.0)
- added Q9: 2N7002, Package_TO_SOT_SMD:SOT-23, F.Cu at (193.8, 52.2)
- added R1: 220R, Resistor_SMD:R_0805_2012Metric_Pad1.20x1.40mm_HandSolder, F.Cu at (214.2, 57.9)
- added R10: 10k, Resistor_SMD:R_0805_2012Metric_Pad1.20x1.40mm_HandSolder, F.Cu at (185.6, 89.5)
- added R11: 10k, Resistor_SMD:R_0805_2012Metric_Pad1.20x1.40mm_HandSolder, F.Cu at (185.6, 92.4)
- added R12: 10k, Resistor_SMD:R_0805_2012Metric_Pad1.20x1.40mm_HandSolder, F.Cu at (185.6, 95.3)
- added R13: 220R, Resistor_SMD:R_0805_2012Metric_Pad1.20x1.40mm_HandSolder, F.Cu at (199.0, 103.2)
- added R14: 220R, Resistor_SMD:R_0805_2012Metric_Pad1.20x1.40mm_HandSolder, F.Cu at (199.0, 106.2)
- added R15: 10k, Resistor_SMD:R_0805_2012Metric_Pad1.20x1.40mm_HandSolder, F.Cu at (70.2, 90.4)
- added R16: 10k, Resistor_SMD:R_0805_2012Metric_Pad1.20x1.40mm_HandSolder, F.Cu at (70.2, 93.3)
- added R17: 200R, Resistor_SMD:R_0805_2012Metric_Pad1.20x1.40mm_HandSolder, F.Cu at (70.2, 104.2)
- added R18: 10k, Resistor_SMD:R_0805_2012Metric_Pad1.20x1.40mm_HandSolder, F.Cu at (70.2, 107.1)
- added R19: 10k, Resistor_SMD:R_0805_2012Metric_Pad1.20x1.40mm_HandSolder, F.Cu at (70.2, 110.1)
- added R2: 220R, Resistor_SMD:R_0805_2012Metric_Pad1.20x1.40mm_HandSolder, F.Cu at (214.2, 60.9)
- added R20: 10k, Resistor_SMD:R_0805_2012Metric_Pad1.20x1.40mm_HandSolder, F.Cu at (70.2, 113.0)
- added R21: 10k, Resistor_SMD:R_0805_2012Metric_Pad1.20x1.40mm_HandSolder, F.Cu at (220.3, 72.5)
- added R22: 10k, Resistor_SMD:R_0805_2012Metric_Pad1.20x1.40mm_HandSolder, F.Cu at (220.3, 75.4)
- added R23: 10k, Resistor_SMD:R_0805_2012Metric_Pad1.20x1.40mm_HandSolder, F.Cu at (220.3, 78.4)
- added R24: 10k, Resistor_SMD:R_0805_2012Metric_Pad1.20x1.40mm_HandSolder, F.Cu at (220.3, 81.3)
- added R25: 10k, Resistor_SMD:R_0805_2012Metric_Pad1.20x1.40mm_HandSolder, F.Cu at (185.6, 100.3)
- added R26: 10k, Resistor_SMD:R_0805_2012Metric_Pad1.20x1.40mm_HandSolder, F.Cu at (185.6, 103.2)
- added R27: 10k, Resistor_SMD:R_0805_2012Metric_Pad1.20x1.40mm_HandSolder, F.Cu at (185.6, 106.2)
- added R28: 10k, Resistor_SMD:R_0805_2012Metric_Pad1.20x1.40mm_HandSolder, F.Cu at (185.6, 109.2)
- added R29: 10k, Resistor_SMD:R_0805_2012Metric_Pad1.20x1.40mm_HandSolder, F.Cu at (199.0, 86.5)
- added R3: 10k, Resistor_SMD:R_0805_2012Metric_Pad1.20x1.40mm_HandSolder, F.Cu at (214.2, 63.8)
- added R30: 10k, Resistor_SMD:R_0805_2012Metric_Pad1.20x1.40mm_HandSolder, F.Cu at (199.0, 89.5)
- added R31: 10k, Resistor_SMD:R_0805_2012Metric_Pad1.20x1.40mm_HandSolder, F.Cu at (199.0, 92.4)
- added R32: 10k, Resistor_SMD:R_0805_2012Metric_Pad1.20x1.40mm_HandSolder, F.Cu at (199.0, 95.3)
- added R33: 10k, Resistor_SMD:R_0805_2012Metric_Pad1.20x1.40mm_HandSolder, F.Cu at (188.9, 57.9)
- added R34: 220R, Resistor_SMD:R_0805_2012Metric_Pad1.20x1.40mm_HandSolder, F.Cu at (188.9, 60.9)
- added R35: 220R, Resistor_SMD:R_0805_2012Metric_Pad1.20x1.40mm_HandSolder, F.Cu at (188.9, 63.8)
- added R36: 10k, Resistor_SMD:R_0805_2012Metric_Pad1.20x1.40mm_HandSolder, F.Cu at (212.3, 110.8)
- added R37: 220R, Resistor_SMD:R_0805_2012Metric_Pad1.20x1.40mm_HandSolder, F.Cu at (212.3, 113.8)
- added R38: 220R, Resistor_SMD:R_0805_2012Metric_Pad1.20x1.40mm_HandSolder, F.Cu at (212.3, 116.7)
- added R39: 10k, Resistor_SMD:R_0805_2012Metric_Pad1.20x1.40mm_HandSolder, F.Cu at (212.3, 98.7)
- added R4: 180, Resistor_SMD:R_0805_2012Metric_Pad1.20x1.40mm_HandSolder, F.Cu at (70.2, 84.5)
- added R40: 220R, Resistor_SMD:R_0805_2012Metric_Pad1.20x1.40mm_HandSolder, F.Cu at (212.3, 101.6)
- added R41: 220R, Resistor_SMD:R_0805_2012Metric_Pad1.20x1.40mm_HandSolder, F.Cu at (212.3, 104.6)
- added R42: 10k, Resistor_SMD:R_0805_2012Metric_Pad1.20x1.40mm_HandSolder, F.Cu at (214.2, 45.8)
- added R43: 220R, Resistor_SMD:R_0805_2012Metric_Pad1.20x1.40mm_HandSolder, F.Cu at (214.2, 48.7)
- added R44: 220R, Resistor_SMD:R_0805_2012Metric_Pad1.20x1.40mm_HandSolder, F.Cu at (214.2, 51.7)
- added R45: 10k, Resistor_SMD:R_0805_2012Metric_Pad1.20x1.40mm_HandSolder, F.Cu at (212.3, 86.5)
- added R46: 220R, Resistor_SMD:R_0805_2012Metric_Pad1.20x1.40mm_HandSolder, F.Cu at (212.3, 89.5)
- added R47: 220R, Resistor_SMD:R_0805_2012Metric_Pad1.20x1.40mm_HandSolder, F.Cu at (212.3, 92.4)
- added R48: 10k, Resistor_SMD:R_0805_2012Metric_Pad1.20x1.40mm_HandSolder, F.Cu at (188.9, 45.8)
- added R49: 220R, Resistor_SMD:R_0805_2012Metric_Pad1.20x1.40mm_HandSolder, F.Cu at (188.9, 48.7)
- added R5: 180, Resistor_SMD:R_0805_2012Metric_Pad1.20x1.40mm_HandSolder, F.Cu at (70.2, 87.4)
- added R50: 220R, Resistor_SMD:R_0805_2012Metric_Pad1.20x1.40mm_HandSolder, F.Cu at (188.9, 51.7)
- added R51: 10k, Resistor_SMD:R_0805_2012Metric_Pad1.20x1.40mm_HandSolder, F.Cu at (201.6, 45.8)
- added R52: 220R, Resistor_SMD:R_0805_2012Metric_Pad1.20x1.40mm_HandSolder, F.Cu at (201.6, 48.7)
- added R53: 220R, Resistor_SMD:R_0805_2012Metric_Pad1.20x1.40mm_HandSolder, F.Cu at (201.6, 51.7)
- added R54: 10k, Resistor_SMD:R_0805_2012Metric_Pad1.20x1.40mm_HandSolder, F.Cu at (201.6, 57.9)
- added R55: 220R, Resistor_SMD:R_0805_2012Metric_Pad1.20x1.40mm_HandSolder, F.Cu at (201.6, 60.9)
- added R56: 220R, Resistor_SMD:R_0805_2012Metric_Pad1.20x1.40mm_HandSolder, F.Cu at (201.6, 63.8)
- added R6: 10k, Resistor_SMD:R_0805_2012Metric_Pad1.20x1.40mm_HandSolder, F.Cu at (199.0, 100.3)
- added R7: 200R, Resistor_SMD:R_0805_2012Metric_Pad1.20x1.40mm_HandSolder, F.Cu at (70.2, 98.3)
- added R8: 200R, Resistor_SMD:R_0805_2012Metric_Pad1.20x1.40mm_HandSolder, F.Cu at (70.2, 101.2)
- added R9: 10k, Resistor_SMD:R_0805_2012Metric_Pad1.20x1.40mm_HandSolder, F.Cu at (185.6, 86.5)
- added SENS1: MTSW-103-23-F-D-230, MTSW-103-23-F-D-230:SAMTEC_MTSW-103-23-F-D-230, F.Cu at (57.4, 86.6)
- added SENS2: MTSW-103-23-F-D-230, MTSW-103-23-F-D-230:SAMTEC_MTSW-103-23-F-D-230, F.Cu at (57.4, 93.2)
- added SENS3: MTSW-103-23-F-D-230, MTSW-103-23-F-D-230:SAMTEC_MTSW-103-23-F-D-230, F.Cu at (57.4, 99.9)
- added SENS4: MTSW-103-23-F-D-230, MTSW-103-23-F-D-230:SAMTEC_MTSW-103-23-F-D-230, F.Cu at (57.4, 106.5)
- added SPI1: MTSW-103-23-F-D-230, MTSW-103-23-F-D-230:SAMTEC_MTSW-103-23-F-D-230, F.Cu at (186.7, 117.8)
- added U1: SN74LVC2G14DBV, Package_TO_SOT_SMD:SOT-23-6, F.Cu at (227.1, 58.9)
- added U10: ITR8307-S17-TR8, OptoDevice:Everlight_ITR1201SR10AR, F.Cu at (79.7, 100.4)
- added U11: ITR8307-S17-TR8, OptoDevice:Everlight_ITR1201SR10AR, F.Cu at (87.0, 103.0)
- added U12: VL53L0CXV0DH1, Sensor_Distance:ST_VL53L1x, F.Cu at (204.7, 87.2)
- added U13: TB6612FNG, Package_SO:SSOP-24_5.3x8.2mm_P0.65mm, F.Cu at (193.3, 76.0)
- added U2: TB6612FNG, Package_SO:SSOP-24_5.3x8.2mm_P0.65mm, F.Cu at (210.7, 76.0)
- added U3: VL53L0CXV0DH1, Sensor_Distance:ST_VL53L1x, F.Cu at (226.1, 73.2)
- added U4: ATMEGA328P-AU, ATMEGA328P-AU:QFP80P900X900X120-32N, F.Cu at (100.5, 78.5)
- added U5: VL53L0CXV0DH1, Sensor_Distance:ST_VL53L1x, F.Cu at (191.4, 87.2)
- added U6: VL53L0CXV0DH1, Sensor_Distance:ST_VL53L1x, F.Cu at (191.4, 101.0)
- added U7: LM1117S-5.0, Package_TO_SOT_SMD:TO-263-3_TabPin2, F.Cu at (78.5, 47.4)
- added U8: ITR8307-S17-TR8, OptoDevice:Everlight_ITR1201SR10AR, F.Cu at (74.9, 100.4)
- added U9: LM1117S-3.3, Package_TO_SOT_SMD:TO-263-3_TabPin2, F.Cu at (78.5, 59.8)
- added Y1: ECS-160-20-4DN, ECS-160-20-4DN:XTAL_ECS-160-20-4DN, F.Cu at (63.0, 69.5)
Other:
- board outline added: 90 x 90 mm

Commit message: chyba gotowy schemat
Parts:
- removed C19, C20: 10nF, Capacitor_SMD:C_0805_2012Metric_Pad1.18x1.45mm_HandSolder
- removed C23: 10uF, Capacitor_SMD:C_0805_2012Metric_Pad1.18x1.45mm_HandSolder
- removed D1, D10, D11, D12, D4, D9: blue, LED_THT:LED_D3.0mm
- removed J2: Conn_01x02_Pin, Connector_JST:JST_EH_B2B-EH-A_1x02_P2.50mm_Vertical
- removed Q10, Q11, Q2, Q3, Q8, Q9: 2N7002, Package_TO_SOT_SMD:SOT-23
- removed R48, R51, R54: 10k, Resistor_SMD:R_0805_2012Metric_Pad1.20x1.40mm_HandSolder
- removed R49, R50, R52, R53, R55, R56: 220R, Resistor_SMD:R_0805_2012Metric_Pad1.20x1.40mm_HandSolder
- removed U13: TB6612FNG, Package_SO:SSOP-24_5.3x8.2mm_P0.65mm
- added C27: 10uF, Capacitor_SMD:C_0805_2012Metric_Pad1.18x1.45mm_HandSolder, B.Cu at (141.0, 69.0)
- added C28: 10nF, Capacitor_SMD:C_0805_2012Metric_Pad1.18x1.45mm_HandSolder, B.Cu at (138.0, 69.0)
- added C29: 10nF, Capacitor_SMD:C_0805_2012Metric_Pad1.18x1.45mm_HandSolder, B.Cu at (135.0, 69.0)
- added C30: 10uF, Capacitor_SMD:C_0805_2012Metric_Pad1.18x1.45mm_HandSolder, B.Cu at (132.0, 69.0)
- added M1: ~, Motors_KoNaR:KoNaR_Motor, F.Cu at (171.5, 116.0)
- added M2: ~, Motors_KoNaR:KoNaR_Motor, F.Cu at (130.5, 116.0)
- added U14: TB6612FNG, Package_SO:SSOP-24_5.3x8.2mm_P0.65mm, B.Cu at (138.0, 115.5)
- C1, C10, C11, C12, C13, C2, C24, C25, C26, C3, C4, C5, C6, C8, C9, D2, D3, R15, R16, R17, R18, R19, R20, R21, R22, R23, R24, R4, R5, R7, R8, U2, U3, U8: moved to B.Cu
- C18: value 10uF -> 100nF; moved to B.Cu
- R1, R47: value 220R -> 10k; moved to B.Cu
- R13: value 220R -> 10k
- R14, R46: value 220R -> 20k
- R2: value 220R -> 20k; moved to B.Cu
- R6: value 10k -> 20k
- moved SENS4 140.9 mm to (194.5, 73.9), turned to -90 degrees
- moved R7 127.7 mm to (194.5, 69.0), turned to 90 degrees
- moved U9 126.5 mm to (174.7, 142.0)
- moved R8 125.5 mm to (191.5, 69.0), turned to 90 degrees
- moved SENS3 125.1 mm to (174.4, 55.5)
- moved R17 123.5 mm to (188.6, 69.0), turned to 90 degrees
- moved R18 121.5 mm to (185.6, 69.0), turned to 90 degrees
- moved R19 119.7 mm to (182.7, 69.0), turned to 90 degrees
- moved R20 118.0 mm to (179.7, 69.0), turned to 90 degrees
- moved U11 115.8 mm to (195.1, 61.5), turned to 90 degrees
- moved C1 114.5 mm to (183.1, 88.9), turned to 90 degrees
- moved C2 111.1 mm to (180.1, 88.9), turned to 90 degrees
- moved R4 106.7 mm to (176.9, 84.1), turned to 90 degrees
- moved U7 106.2 mm to (126.8, 142.0), turned to 180 degrees
- moved Q1 106.0 mm to (157.5, 141.6), turned to 90 degrees
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Connections:
- net /uC/XTAL1 renamed XTAL1
- net /uC/XTAL2 renamed XTAL2
- B1 pad 1: GND -> /programming_connector/RST
- C13 pad 1: +3V3 -> +5V
- C8 pad 1: +3V3 -> +5V
- Q4 pad 2: /converter_GPIO1_4/STX -> GPIO1_4
- Q4 pad 3: GPIO1_4 -> /converter_GPIO1_4/STX
- Q5 pad 2: /converter_GPIO1_4/STX -> GPIO1_3
- Q5 pad 3: GPIO1_3 -> /converter_GPIO1_3/STX
- Q6 pad 2: /converter_GPIO1_2/STX -> GPIO1_2
- Q6 pad 3: GPIO1_2 -> /converter_GPIO1_2/STX
- Q7 pad 2: /converter_GPIO1_1/STX -> GPIO1_1
- Q7 pad 3: GPIO1_1 -> /converter_GPIO1_1/STX
- R1 pad 1: Net-(D1-K) -> Net-(U3-XSHUT)
- R1 pad 2: /converter_SDA/STX -> XSHUT_2
- R10 pad 2: /converter_SCL/STX -> SCL
- R11 pad 2: /converter_SDA/STX -> SDA
- R12 pad 2: /sensor1/GPIO1 -> /converter_GPIO1_1/STX
- R13 pad 1: +3V3 -> Net-(U12-XSHUT)
- R13 pad 2: Net-(Q3-G) -> XSHUT_3
- R14 pad 1: Net-(D4-K) -> GND
- R14 pad 2: /converter_SCL/STX -> Net-(U12-XSHUT)
- R2 pad 1: +3V3 -> GND
- R2 pad 2: Net-(Q2-G) -> Net-(U3-XSHUT)
- R21 pad 1: +3V3 -> +5V
- R21 pad 2: /sensor2/XSHUT -> Net-(U3-XSHUT)
- R22 pad 1: +3V3 -> +5V
- R22 pad 2: /converter_SCL/STX -> SCL
- R23 pad 1: +3V3 -> +5V
- R23 pad 2: /converter_SDA/STX -> SDA
- R24 pad 1: +3V3 -> +5V
- R24 pad 2: /sensor2/GPIO1 -> /converter_GPIO1_2/STX
- R25 pad 2: /sensor3/XSHUT -> Net-(U6-XSHUT)
- R26 pad 2: /converter_SCL/STX -> SCL
- R27 pad 2: /converter_SDA/STX -> SDA
- R28 pad 2: /sensor3/GPIO1 -> /converter_GPIO1_3/STX
- R29 pad 2: /sensor4/XSHUT -> Net-(U12-XSHUT)
- R3 pad 1: +5V -> Net-(U6-XSHUT)
- R3 pad 2: SDA -> XSHUT_4
- R30 pad 2: /converter_SCL/STX -> SCL
- R31 pad 2: /converter_SDA/STX -> SDA
- R32 pad 2: /sensor4/GPIO1 -> /converter_GPIO1_4/STX
- R33 pad 2: GPIO1_4 -> /converter_GPIO1_4/STX
- R35 pad 2: /converter_GPIO1_4/STX -> GPIO1_4
- R36 pad 2: GPIO1_3 -> /converter_GPIO1_3/STX
- R38 pad 2: /converter_GPIO1_4/STX -> GPIO1_3
- R39 pad 2: GPIO1_2 -> /converter_GPIO1_2/STX
- R41 pad 2: /converter_GPIO1_2/STX -> GPIO1_2
- R42 pad 2: GPIO1_1 -> /converter_GPIO1_1/STX
- R44 pad 2: /converter_GPIO1_1/STX -> GPIO1_1
- R45 pad 1: +5V -> Net-(U5-XSHUT)
- R46 pad 1: +3V3 -> GND
- R46 pad 2: Net-(Q8-G) -> Net-(U5-XSHUT)
- R47 pad 1: Net-(D9-K) -> /programming_connector/RST
- R47 pad 2: /converter_XSHUT_1/STX -> +5V
- R6 pad 1: +5V -> GND
- R6 pad 2: SCL -> Net-(U6-XSHUT)
- R9 pad 2: /sensor1/XSHUT -> Net-(U5-XSHUT)
- SPI1 pad 01: GND -> /programming_connector/MISO
- SPI1 pad 06: /programming_connector/MISO -> GND
- U1 pad 1: /inverter/DIR2_2 -> /inverter/DIR1_1
- U1 pad 4: /inverter/DIR1_1 -> /inverter/DIR2_2
- U12 pad 10: /converter_SCL/STX -> SCL
- U12 pad 5: /sensor4/XSHUT -> Net-(U12-XSHUT)
- U12 pad 7: /sensor4/GPIO1 -> /converter_GPIO1_4/STX
- U12 pad 9: /converter_SDA/STX -> SDA
- U2 pad 1: unconnected-(U2-AO1-Pad1) -> Net-(M1-Pad2)
- U2 pad 11: unconnected-(U2-AO1-Pad1) -> Net-(M1-Pad2)
- U2 pad 12: unconnected-(U2-AO1-Pad1) -> Net-(M1-Pad2)
- U2 pad 16: /motor_driver1/DIR2 -> /inverter/DIR2_1
- U2 pad 17: /motor_driver1/DIR1 -> /inverter/DIR1_1
- U2 pad 2: unconnected-(U2-AO1-Pad1) -> Net-(M1-Pad2)
- U2 pad 21: /motor_driver1/DIR1 -> /inverter/DIR1_1
- U2 pad 22: /motor_driver1/DIR2 -> /inverter/DIR2_1
- U2 pad 5: unconnected-(U2-AO2-Pad5) -> Net-(M1-Pad1)
- U2 pad 6: unconnected-(U2-AO2-Pad5) -> Net-(M1-Pad1)
- U2 pad 7: unconnected-(U2-AO2-Pad5) -> Net-(M1-Pad1)
- U2 pad 8: unconnected-(U2-AO2-Pad5) -> Net-(M1-Pad1)
- U3 pad 1: +3V3 -> +5V
- U3 pad 10: /converter_SCL/STX -> SCL
- U3 pad 11: +3V3 -> +5V
- U3 pad 5: /sensor2/XSHUT -> Net-(U3-XSHUT)
- U3 pad 7: /sensor2/GPIO1 -> /converter_GPIO1_2/STX
- U3 pad 9: /converter_SDA/STX -> SDA
- U4 pad 10: /uC/PWM2 -> /motor_driver2/PWM2
- U4 pad 12: /line_sensors/LS1 -> GPIO1_1
- U4 pad 13: /line_sensors/LS3 -> GPIO1_2
- U4 pad 14: /line_sensors/LS2 -> GPIO1_3
- U4 pad 17: unconnected-(U4-PB5-Pad17) -> /programming_connector/SCK
- U4 pad 23: GPIO1_1 -> /line_sensors/LS1
- U4 pad 24: GPIO1_2 -> /line_sensors/LS3
- U4 pad 25: GPIO1_3 -> /line_sensors/LS2
- U5 pad 10: /converter_SCL/STX -> SCL
- U5 pad 5: /sensor1/XSHUT -> Net-(U5-XSHUT)
- U5 pad 7: /sensor1/GPIO1 -> /converter_GPIO1_1/STX
- U5 pad 9: /converter_SDA/STX -> SDA
- U6 pad 10: /converter_SCL/STX -> SCL
- U6 pad 5: /sensor3/XSHUT -> Net-(U6-XSHUT)
- U6 pad 7: /sensor3/GPIO1 -> /converter_GPIO1_3/STX
- U6 pad 9: /converter_SDA/STX -> SDA
Other:
- board size 90 x 90 mm -> 100 x 100 mm
- rule pad_to_mask_clearance: 0.038 -> 0

Commit message: stan przed usunięciem jednego czujnika lini
Parts:
- removed C11, C12: 10uF, Capacitor_SMD:C_0805_2012Metric_Pad1.18x1.45mm_HandSolder
- removed C13, C15, C17, C22: 4,7uF, Capacitor_SMD:C_0805_2012Metric_Pad1.18x1.45mm_HandSolder
- removed C14, C16, C21, C8: 100nF, Capacitor_SMD:C_0805_2012Metric_Pad1.18x1.45mm_HandSolder
- removed D5, D6, D7, D8: blue, LED_THT:LED_D3.0mm
- removed Q4, Q5, Q6, Q7: 2N7002, Package_TO_SOT_SMD:SOT-23
- removed R1, R10, R11, R12, R13, R21, R22, R23, R24, R25, R26, R27, R28, R29, R3, R30, R31, R32, R33, R36, R39, R42, R45, R9: 10k, Resistor_SMD:R_0805_2012Metric_Pad1.20x1.40mm_HandSolder
- removed R14, R2, R46, R6: 20k, Resistor_SMD:R_0805_2012Metric_Pad1.20x1.40mm_HandSolder
- removed R34, R35, R37, R38, R40, R41, R43, R44: 220R, Resistor_SMD:R_0805_2012Metric_Pad1.20x1.40mm_HandSolder
- removed SENS1, SENS2, SENS3, SENS4: MTSW-103-23-F-D-230, MTSW-103-23-F-D-230:SAMTEC_MTSW-103-23-F-D-230
- removed U12, U3, U5, U6: VL53L0CXV0DH1, Sensor_Distance:ST_VL53L1x
- removed U9: LM1117S-3.3, Package_TO_SOT_SMD:TO-263-3_TabPin2
- added SPI2: MTSW-103-23-F-D-230, MTSW-103-23-F-D-230:SAMTEC_MTSW-103-23-F-D-230, F.Cu at (55.4, 68.0)
- added SPI3: MTSW-103-23-F-D-230, MTSW-103-23-F-D-230:SAMTEC_MTSW-103-23-F-D-230, F.Cu at (70.7, 54.8)
- added SPI4: MTSW-103-23-F-D-230, MTSW-103-23-F-D-230:SAMTEC_MTSW-103-23-F-D-230, F.Cu at (124.0, 54.5)
- added SPI5: MTSW-103-23-F-D-230, MTSW-103-23-F-D-230:SAMTEC_MTSW-103-23-F-D-230, F.Cu at (140.0, 68.0)
- C1, C18, C2, C24, C25, C26, D2, D3, R15, R16, R17, R18, R19, R20, R4, R47, R5, R7, R8, U8: moved to F.Cu
- C10, C27, C30, C4, C5, C9: footprint Capacitor_SMD:C_0805_2012Metric_Pad1.18x1.45mm_HandSolder -> Capacitor_Tantalum_SMD:CP_EIA-3528-12_Kemet-T
- Q1, U7: moved to B.Cu
- moved U10 114.9 mm to (220.2, 74.0), turned to 0 degrees
- moved U1 97.8 mm to (222.6, 129.7)
- moved C7 97.8 mm to (222.4, 133.4)
- moved U8 97.5 mm to (215.4, 74.0), turned to 0 degrees
- moved J1 80.6 mm to (100.0, 90.5)
- moved Q1 77.9 mm to (103.0, 86.0), turned to 180 degrees
- moved Y1 77.4 mm to (224.4, 97.6), turned to 0 degrees
- moved C4 76.6 mm to (82.5, 101.2), turned to -90 degrees
- moved C5 76.5 mm to (82.5, 106.7), turned to -90 degrees
- moved C3 76.0 mm to (84.5, 97.2), turned to 0 degrees
- moved U7 73.4 mm to (88.8, 79.3)
- moved C6 71.5 mm to (86.4, 108.5), turned to 0 degrees
- moved D3 68.2 mm to (231.7, 109.0), turned to 0 degrees
- moved D2 60.8 mm to (231.7, 103.5), turned to 0 degrees
- moved C9 57.3 mm to (102.9, 82.0), turned to 0 degrees
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Connections:
- net Net-(M1-Pad1) renamed /motor_driver1/MOTOR_IN2
- net Net-(M1-Pad2) renamed /motor_driver1/MOTOR_IN1
- net Net-(M2-Pad1) renamed /motor_driver2/MOTOR_IN2
- net Net-(M2-Pad2) renamed /motor_driver2/MOTOR_IN1
- B1 pad 1: /programming_connector/RST -> GND
- B1 pad 2: Net-(U4-PC6/~{RESET}) -> /programming_connector/RST
- U1 pad 1: /inverter/DIR1_1 -> /inverter/DIRB_1
- U1 pad 3: /inverter/DIR1_2 -> /inverter/DIRB_2
- U1 pad 4: /inverter/DIR2_2 -> /inverter/DIRA_2
- U1 pad 6: /inverter/DIR2_1 -> /inverter/DIRA_1
- U14 pad 16: /inverter/DIR2_2 -> /inverter/DIRB_2
- U14 pad 17: /inverter/DIR1_2 -> /inverter/DIRA_2
- U14 pad 21: /inverter/DIR1_2 -> /inverter/DIRA_2
- U14 pad 22: /inverter/DIR2_2 -> /inverter/DIRB_2
- U2 pad 16: /inverter/DIR2_1 -> /inverter/DIRB_1
- U2 pad 17: /inverter/DIR1_1 -> /inverter/DIRA_1
- U2 pad 21: /inverter/DIR1_1 -> /inverter/DIRA_1
- U2 pad 22: /inverter/DIR2_1 -> /inverter/DIRB_1
- U4 pad 1: XSHUT_4 -> /sensor4/X4
- U4 pad 11: /inverter/DIR2_2 -> /inverter/DIRB_2
- U4 pad 12: GPIO1_1 -> /sensor1/G1
- U4 pad 13: GPIO1_2 -> /sensor2/G2
- U4 pad 14: GPIO1_3 -> /sensor3/G3
- U4 pad 2: /inverter/DIR1_2 -> /inverter/DIRB_1
- U4 pad 26: GPIO1_4 -> /sensor4/G4
- U4 pad 27: SDA -> /sensor1/SDA
- U4 pad 28: SCL -> /sensor1/SCL
- U4 pad 29: Net-(U4-PC6/~{RESET}) -> /programming_connector/RST
- U4 pad 30: XSHUT_1 -> /sensor1/X1
- U4 pad 31: XSHUT_2 -> /sensor2/X2
- U4 pad 32: XSHUT_3 -> /sensor3/X3
