File: Warsztaty/minisumo/minisumo_pcb/minisumo_pcb.kicad_pcb (KiCad board)
At the start: 2 copper layers, 76.7 x 88 mm, 61 parts, among them J2 MTSW-103-23-F-S-235, M1 HTSW-102-08-L-S, M2 HTSW-102-08-L-S, Q1 PMOS, U7 LM1117S-5.0, Y1 ECS-160-20-4DN

Commit message: ostateczna wersja płytki
Parts:
- C25, C26: moved to B.Cu
- moved C25 8.33 mm to (130.2, 104.2), turned to -45 degrees
- moved C26 7.67 mm to (126.3, 104.2), turned to -135 degrees
- moved C9 0.38 mm to (119.9, 75.1)
- moved C10 0.37 mm to (126.6, 78.4)
- moved ES3 0.06 mm to (139.0, 113.3)
Routing:
- net +5V: track 312.1 -> 305.8 mm, vias 8 -> 5
- net GND: track 47.2 -> 49.9 mm
- net /inverter/DIRB_2: track 65.2 -> 64.5 mm
- net /programming_connector/RST: track 53.9 -> 54.5 mm
- net /line_sensors/LS2: track 58.9 -> 59.4 mm
Other:
- board size 76.7 x 88 mm -> 76.8 x 88 mm
